File: hardware/v3/SAX_3.sch (KiCad schematic (older format))
At the start: 81 parts, among them J1 joystick, J2 LED strip, J3 SSD1306 SPI, J4 MIDI OUT Y:M5 - R:M4, J5 Batt, J6 Neck - Y:O BK:B R:3.3, J7 Conn_01x03_Female, J8 MXP5010, U1 74HC165, U2 74HC165, U3 74HC165, U4 Teensy3.2_breadboard_friendly

Commit message: Updated PCB with correct JST connectors, optimized PCB
Parts:
- J5: footprint Connector_JST:JST_PH_B2B-PH-K_1x02_P2.00mm_Vertical -> Connector_JST:JST_EH_B2B-EH-A_1x02_P2.50mm_Vertical
Changed lines of the file:
@@
 F 0 "J5" H 10578 2276 50  0000 L CNN
 F 1 "Batt" H 10578 2185 50  0000 L CNN
-F 2 "Connector_JST:JST_PH_B2B-PH-K_1x02_P2.00mm_Vertical" H 10550 2300 50  0001 C CNN
+F 2 "Connector_JST:JST_EH_B2B-EH-A_1x02_P2.50mm_Vertical" H 10550 2300 50  0001 C CNN
 F 3 "~" H 10550 2300 50  0001 C CNN
 	1    10550 2300

Commit message: Updated PCB
Parts:
- added H1, H2: MountingHole, MountingHole:MountingHole_4.3mm_M4_DIN965_Pad, symbol Mechanical:MountingHole
- added H3, H4, H5: MountingHole, MountingHole:MountingHole_3.2mm_M3_DIN965_Pad, symbol Mechanical:MountingHole
Changed lines of the file:
@@
 	0    1    1    0
 $EndComp
+$Comp
+L Mechanical:MountingHole H1
+U 1 1 61CA7701
+P 9500 4650
+F 0 "H1" H 9600 4696 50  0000 L CNN
+F 1 "MountingHole" H 9600 4605 50  0000 L CNN
+F 2 "MountingHole:MountingHole_4.3mm_M4_DIN965_Pad" H 9500 4650 50  0001 C CNN
+F 3 "~" H 9500 4650 50  0001 C CNN
+	1    9500 4650
+	1    0    0    -1
+$EndComp
+$Comp
+L Mechanical:MountingHole H3
+U 1 1 61CA8909
+P 10000 4650
+F 0 "H3" H 10100 4696 50  0000 L CNN
+F 1 "MountingHole" H 10100 4605 50  0000 L CNN
+F 2 "MountingHole:MountingHole_3.2mm_M3_DIN965_Pad" H 10000 4650 50  0001 C CNN
+F 3 "~" H 10000 4650 50  0001 C CNN
+	1    10000 4650
+	1    0    0    -1
+$EndComp
+$Comp
+L Mechanical:MountingHole H2
+U 1 1 61CA9906
+P 9500 4950
+F 0 "H2" H 9600 4996 50  0000 L CNN
+F 1 "MountingHole" H 9600 4905 50  0000 L CNN
+F 2 "MountingHole:MountingHole_4.3mm_M4_DIN965_Pad" H 9500 4950 50  0001 C CNN
+F 3 "~" H 9500 4950 50  0001 C CNN
+	1    9500 4950
+	1    0    0    -1
+$EndComp
+$Comp
+L Mechanical:MountingHole H4
+U 1 1 61CA990C
+P 10000 4950
+F 0 "H4" H 10100 4996 50  0000 L CNN
+F 1 "MountingHole" H 10100 4905 50  0000 L CNN
+F 2 "MountingHole:MountingHole_3.2mm_M3_DIN965_Pad" H 10000 4950 50  0001 C CNN
+F 3 "~" H 10000 4950 50  0001 C CNN
+	1    10000 4950
+	1    0    0    -1
+$EndComp
+$Comp
+L Mechanical:MountingHole H5
+U 1 1 61CC6588
+P 9400 5450
+F 0 "H5" H 9500 5496 50  0000 L CNN
+F 1 "MountingHole" H 9500 5405 50  0000 L CNN
+F 2 "MountingHole:MountingHole_3.2mm_M3_DIN965_Pad" H 9400 5450 50  0001 C CNN
+F 3 "~" H 9400 5450 50  0001 C CNN
+	1    9400 5450
+	1    0    0    -1
+$EndComp
 $EndSCHEMATC
