File: hardware/v3d1/SAX_3.kicad_sch (KiCad schematic)
At the start: 86 parts, among them J1 joystick, J2 LED strip, J3 SSD1306 SPI, J4 MIDI OUT Y:M5 - R:M4, J5 Batt, J6 Neck - Y:O BK:B R:3.3, J7 Conn_01x03_Female, J8 MXP5010, U1 74HC165, U2 74HC165, U3 74HC165, U4 Teensy3.2_breadboard_friendly

Commit message: Update
Parts:
- J5: footprint Connector_JST:JST_EH_B2B-EH-A_1x02_P2.50mm_Vertical -> (none)
Changed lines of the file:
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@@
       (effects (font (size 1.27 1.27)) (justify left))
     )
-    (property "Footprint" "Connector_JST:JST_EH_B2B-EH-A_1x02_P2.50mm_Vertical" (id 2) (at 267.97 58.42 0)
+    (property "Footprint" "" (id 2) (at 267.97 58.42 0)
       (effects (font (size 1.27 1.27)) hide)
     )
@@
     )
     (path "/00000000-0000-0000-0000-000061bf481a"
-      (reference "J5") (unit 1) (value "Batt") (footprint "Connector_JST:JST_EH_B2B-EH-A_1x02_P2.50mm_Vertical")
+      (reference "J5") (unit 1) (value "Batt") (footprint "Connector_JST:JST_XH_B2B-XH-A_1x02_P2.50mm_Vertical")
     )
     (path "/00000000-0000-0000-0000-000061e7f82b"
