File: hardware/v4d2_pico/v4d2_pico.kicad_pcb (KiCad board)
At the start: 2 copper layers, 109 parts, among them J1 joystick, J10 ON/OFF, J11 MIDI IN bk: 5 R: 4, J12 Rvar, J2 LED strip, J3 SSD1306 SPI, J4 MIDI OUT Y:M5 - R:M4, J5 Batt, J6 Neck - O:bk, breath:red, Vcc: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, J7 Conn_01x04_Female, J8 MXP5010, J9 Thumb, Q1 2N7000, SW1 SW_DIP_x01, U1 74HC165, U2 74HC165, U3 74HC165, U4 Pico, U5 FJ08K, U6 6N138, U7 MCP3002

Commit message: Routed PCB
Parts:
- added R28: 10k, Resistor_SMD:R_1206_3216Metric_Pad1.30x1.75mm_HandSolder, F.Cu at (235.6, 33.8)
- added R29: 10k, Resistor_SMD:R_1206_3216Metric_Pad1.30x1.75mm_HandSolder, F.Cu at (235.6, 31.0)
- added U8: CAT24C256, Package_DIP:DIP-8_W7.62mm_Socket, F.Cu at (231.0, 26.9)
- moved TP34 3.56 mm to (241.2, 32.8)
- moved owl_beak 2.50 mm to (187.1, 50.0)
- moved J7 1.55 mm to (174.1, 49.5)
Connections:
- U4 pad 19: unconnected-(U4-Pad19) -> Net-(R28-Pad1)
- U4 pad 20: unconnected-(U4-Pad20) -> Net-(R29-Pad2)
Routing:
- net GND: track 0.00 -> 269.8 mm, vias 0 -> 4
- net ADC_VREF: track 0.00 -> 262.2 mm, vias 0 -> 3
- net ADC_DIN: track 0.00 -> 141.6 mm, vias 0 -> 3
- net Net-(R2-Pad1): track 0.00 -> 133.6 mm, vias 0 -> 6
- net ADC_DOUT: track 0.00 -> 117.2 mm, vias 0 -> 3
- net /SR_CLK: track 0.00 -> 111.1 mm, vias 0 -> 3
- net Net-(R15-Pad1): track 0.00 -> 108.8 mm, vias 0 -> 3
- net Net-(R7-Pad1): track 0.00 -> 107.4 mm, vias 0 -> 1
- net +5V: track 0.00 -> 96.6 mm
- net Net-(R8-Pad1): track 0.00 -> 96.6 mm, vias 0 -> 5
- net Net-(U2-Pad10): track 0.00 -> 96.4 mm, vias 0 -> 10
- net Net-(R26-Pad2): track 0.00 -> 94.9 mm, vias 0 -> 1
- net Net-(R9-Pad1): track 0.00 -> 80.1 mm, vias 0 -> 3
- net Net-(R1-Pad1): track 0.00 -> 79.0 mm, vias 0 -> 2
- net ADC_CLK: track 0.00 -> 77.7 mm, vias 0 -> 4
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- added copper zone on B.Cu, net GND
- added copper zone on F.Cu, net GND
- added copper zone on B.Cu, net Net-(C4-Pad1)
- added copper zone on F.Cu, net Net-(C4-Pad1)
- added copper zone on B.Cu, net Net-(J9-Pad1)
- added copper zone on F.Cu, net Net-(J9-Pad1)
Other:
- board outline added: 86.4 x 94.5 mm
- board text removed: "TES - eSax v4.2 One sided beak With bite pressure"

Commit message: Updated PCB, gerber export
Parts:
- moved owl_small_pcb 2.88 mm to (241.7, 22.9)
Routing:
- net /SR_CLK: track 111.1 -> 110.5 mm
Other:
- board size 86.4 x 94.5 mm -> 86.1 x 94.2 mm
- board text added: "39mm"
- board text added: "Bite"
- board text added: "EEPROM"
- board text added: "Hello there!"
- board text added: "TES sax v4.2 SPI SSD1306 NeoPixel RP2040"
- board text added: "{dblquote}If the emperor looks naked, the emperor IS naked…{dblquote}"
- board text removed: "39mm 10 stripes diam 1mm"
- board text removed: "Rvar-Bite"
- board text removed: "TES sax v4 SPI SSD1306 LED strip RP2040"

Commit message: Updated PCB for v4.2
Parts:
- added C7: 100n, Capacitor_THT:C_Axial_L3.8mm_D2.6mm_P7.50mm_Horizontal, F.Cu at (213.6, 84.1)
- moved owl_big_pcb 7.56 mm to (222.8, 50.2)
- moved R26 3.79 mm to (213.5, 87.8), turned to 0 degrees
Routing:
- net /SR_SH: track 66.3 -> 199.0 mm, vias 2 -> 6
- net ADC_DIN: track 141.6 -> 68.8 mm, vias 3 -> 0
- net Net-(U2-Pad10): track 96.4 -> 37.5 mm, vias 10 -> 4
- net /SR_CLK: track 110.5 -> 61.8 mm
- net Net-(R2-Pad1): track 134.0 -> 86.4 mm, vias 6 -> 3
- net ADC_VREF: track 262.2 -> 300.5 mm, vias 3 -> 2
- net Net-(R18-Pad1): track 74.2 -> 111.7 mm
- net ADC_DOUT: track 117.4 -> 90.6 mm
- net Net-(R26-Pad2): track 94.9 -> 69.8 mm, vias 1 -> 0
- net Net-(J2-Pad1): track 39.9 -> 64.2 mm, vias 3 -> 4
- net Net-(R5-Pad1): track 68.9 -> 89.7 mm, vias 1 -> 3
- net GND: track 269.8 -> 249.7 mm, vias 4 -> 2
- net Net-(R15-Pad1): track 109.1 -> 128.7 mm, vias 3 -> 1
- net +5V: track 96.6 -> 114.5 mm
- net Net-(R11-Pad1): track 73.1 -> 58.8 mm
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Other:
- board size 86.1 x 94.2 mm -> 86.7 x 94.2 mm
- board text added: "SSD1306/ADC: SPI0 DIN: GP3 DOUT: GP4 CLK: GP2 ADC_CS: GP9 SSD_SDA: SSD1306/ADC: SPI0 DIN: GP3 DOUT: GP4 CLK: GP2 ADC_CS: GP9 SSD_RES: GP7 SSD_DC: GP6 SSD_CS: GP5 MIDI IN: GP0 MIDI OUT: GP1 NEOPIXEL: GP21 SHIFT REG: CLK: GP10 SH: GP11 DO: GP12 BREATH: GP26 X/Y: GP27/28"
- board text added: "TES e-SAX v4.2"
