File: hardware/v4d2_pico/v4d2_pico.kicad_sch (KiCad schematic)
At the start: 109 parts, among them J1 joystick, J10 ON/OFF, J11 MIDI IN bk: 5 R: 4, J12 Rvar, J2 LED strip, J3 SSD1306 SPI, J4 MIDI OUT Y:M5 - R:M4, J5 Batt, J6 Neck - O:bk, breath:red, Vcc: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, J7 Conn_01x04_Female, J8 MXP5010, J9 Thumb, Q1 2N7000, SW1 SW_DIP_x01, U1 74HC165, U2 74HC165, U3 74HC165, U4 Pico, U5 FJ08K, U6 6N138, U7 MCP3002, U8 CAT24C256

Commit message: Updated PCB for v4.2
Parts:
- added C7: 100n, Capacitor_THT:C_Axial_L3.8mm_D2.6mm_P7.50mm_Horizontal, symbol Device:C
Connections:
- net +3.3V: now also C7.2
- net GNDA: now also C7.1
Other:
- note removed: "TODO: remove ADC"
Changed lines of the file:
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@@
   (junction (at 184.15 66.548) (diameter 0) (color 0 0 0 0)
   )
+  (junction (at 232.918 114.808) (diameter 0) (color 0 0 0 0)
+  )
   (junction (at 67.31 157.48) (diameter 0) (color 0 0 0 0)
   )
@@
   (junction (at 67.31 104.14) (diameter 0) (color 0 0 0 0)
   )
+  (junction (at 232.918 84.836) (diameter 0) (color 0 0 0 0)
+  )
   (junction (at 49.53 165.1) (diameter 0) (color 0 0 0 0)
   )
@@
     (stroke (width 0) (type default) (color 0 0 0 0))
   )
+  (wire (pts (xy 232.918 114.808) (xy 259.08 114.808))
+    (stroke (width 0) (type default) (color 0 0 0 0))
+  )
   (wire (pts (xy 184.15 76.708) (xy 190.5 76.708))
     (stroke (width 0) (type default) (color 0 0 0 0))
@@
     (stroke (width 0) (type default) (color 0 0 0 0))
   )
+  (wire (pts (xy 232.918 84.836) (xy 238.76 84.836))
+    (stroke (width 0) (type default) (color 0 0 0 0))
+  )
   (wire (pts (xy 359.664 139.7) (xy 364.744 139.7))
     (stroke (width 0) (type default) (color 0 0 0 0))
@@
     (stroke (width 0) (type default) (color 0 0 0 0))
   )
+  (wire (pts (xy 232.918 84.836) (xy 232.918 88.138))
+    (stroke (width 0) (type default) (color 0 0 0 0))
+  )
   (wire (pts (xy 239.268 147.066) (xy 239.268 143.764))
     (stroke (width 0) (type default) (color 0 0 0 0))
@@
     (stroke (width 0) (type default) (color 0 0 0 0))
   )
+  (wire (pts (xy 232.918 117.856) (xy 232.918 114.808))
+    (stroke (width 0) (type default) (color 0 0 0 0))
+  )
   (wire (pts (xy 245.11 125.222) (xy 245.11 145.288))
     (stroke (width 0) (type default) (color 0 0 0 0))
@@
     (stroke (width 0) (type default) (color 0 0 0 0))
   )
+  (wire (pts (xy 246.38 86.106) (xy 246.38 84.836))
+    (stroke (width 0) (type default) (color 0 0 0 0))
+  )
   (wire (pts (xy 72.39 109.22) (xy 68.58 109.22))
     (stroke (width 0) (type default) (color 0 0 0 0))
@@
     (stroke (width 0) (type default) (color 0 0 0 0))
   )
+  (wire (pts (xy 232.918 81.534) (xy 232.918 84.836))
+    (stroke (width 0) (type default) (color 0 0 0 0))
+  )
   (wire (pts (xy 165.1 63.754) (xy 191.516 63.754))
     (stroke (width 0) (type default) (color 0 0 0 0))
@@
     (stroke (width 0) (type default) (color 0 0 0 0))
   )
+  (wire (pts (xy 259.08 114.808) (xy 259.08 86.106))
+    (stroke (width 0) (type default) (color 0 0 0 0))
+  )
   (wire (pts (xy 129.54 41.91) (xy 132.334 41.91))
     (stroke (width 0) (type default) (color 0 0 0 0))
@@
     (stroke (width 0) (type default) (color 0 0 0 0))
   )
+  (wire (pts (xy 232.918 114.808) (xy 232.918 113.538))
+    (stroke (width 0) (type default) (color 0 0 0 0))
+  )
   (wire (pts (xy 154.94 110.236) (xy 154.94 122.936))
     (stroke (width 0) (type default) (color 0 0 0 0))
@@
     (stroke (width 0) (type default) (color 0 0 0 0))
   )
+  (wire (pts (xy 259.08 86.106) (xy 246.38 86.106))
+    (stroke (width 0) (type default) (color 0 0 0 0))
+  )
   (wire (pts (xy 139.192 118.618) (xy 147.32 118.618))
     (stroke (width 0) (type default) (color 0 0 0 0))
@@
     (effects (font (size 1.27 1.27)) (justify left bottom))
   )
-  (text "TODO: remove ADC" (at 198.882 91.948 0)
-    (effects (font (size 1.27 1.27)) (justify left bottom))
-  )
   (text "Beak PCB\n" (at 383.032 100.838 0)
     (effects (font (size 1.27 1.27)) (justify left bottom))
@@
     )
   )
-  (global_label "ADC_VREF" (shape input) (at 232.918 113.538 180) (fields_autoplaced)
+  (global_label "ADC_VREF" (shape input) (at 232.918 117.856 180) (fields_autoplaced)
     (effects (font (size 1.27 1.27)) (justify right))
-    (property "Références Inter-Feuilles" "${INTERSHEET_REFS}" (id 0) (at 221.4014 113.4586 0)
+    (property "Références Inter-Feuilles" "${INTERSHEET_REFS}" (id 0) (at 221.4014 117.7766 0)
       (effects (font (size 1.27 1.27)) (justify right) hide)
     )
@@
     (pin "1")
   )
+  (symbol (lib_id "Device:C") (at 242.57 84.836 90) (unit 1)
+    (in_bom yes) (on_board yes) (fields_autoplaced)
+    (property "Reference" "C7" (id 0) (at 242.57 78.9772 90))
+    (property "Value" "100n" (id 1) (at 242.57 81.5141 90))
+    (property "Footprint" "Capacitor_THT:C_Axial_L3.8mm_D2.6mm_P7.50mm_Horizontal" (id 2) (at 246.38 83.8708 0)
+      (effects (font (size 1.27 1.27)) hide)
+    )
+    (property "Datasheet" "~" (id 3) (at 242.57 84.836 0)
+      (effects (font (size 1.27 1.27)) hide)
+    )
+    (pin "1")
+    (pin "2")
+  )
   (symbol (lib_id "Device:C") (at 359.918 127 0) (unit 1)
     (in_bom yes) (on_board yes) (fields_autoplaced)
@@
     )
   )
-  (symbol (lib_id "power:GNDA") (at 232.918 88.138 180) (unit 1)
+  (symbol (lib_id "power:GNDA") (at 232.918 81.534 180) (unit 1)
     (in_bom yes) (on_board yes) (fields_autoplaced)
-    (property "Reference" "#PWR08" (id 0) (at 232.918 81.788 0)
+    (property "Reference" "#PWR08" (id 0) (at 232.918 75.184 0)
       (effects (font (size 1.27 1.27)) hide)
     )
-    (property "Value" "GNDA" (id 1) (at 232.918 84.5622 0))
-    (property "Footprint" "" (id 2) (at 232.918 88.138 0)
+    (property "Value" "GNDA" (id 1) (at 232.918 77.9582 0))
+    (property "Footprint" "" (id 2) (at 232.918 81.534 0)
       (effects (font (size 1.27 1.27)) hide)
     )
-    (property "Datasheet" "" (id 3) (at 232.918 88.138 0)
+    (property "Datasheet" "" (id 3) (at 232.918 81.534 0)
       (effects (font (size 1.27 1.27)) hide)
     )
@@
       (reference "C6") (unit 1) (value "470p") (footprint "Capacitor_THT:C_Disc_D3.4mm_W2.1mm_P2.50mm")
     )
+    (path "/7855b814-29be-4d86-a237-4e32e8f8ab4f"
+      (reference "C7") (unit 1) (value "100n") (footprint "Capacitor_THT:C_Axial_L3.8mm_D2.6mm_P7.50mm_Horizontal")
+    )
     (path "/6ea2bc83-6e60-44b0-9fd6-b93a1503a50c"
